File: electronics/v1/v1.sch (KiCad schematic (older format))
At the start: 47 parts, among them J1 AVR-ISP-6, J2 SENSE_ELECTRODE, U1 ATmega328P-MMH, U2 MCP16251T-I/CH, U3 AT42QT1010-TSHR, Y1 8MHz

Commit message: Nearly finished board but realized I used 0603 *metric*, not *imperial*. Will change.
Parts:
- C1, C2, CIN1, COUT1: footprint Capacitor_SMD:C_0201_0603Metric -> Capacitor_SMD:C_0603_1608Metric
- CS1: footprint Capacitor_SMD:C_0201_0603Metric -> Capacitor_SMD:C_1206_3216Metric_Pad1.42x1.75mm_HandSolder
- D1, D10, D11, D12, D13, D14, D15, D16, D17, D18, D19, D2, D20, D21, D22, D23, D24, D3, D4, D5, D6, D7, D8, D9: footprint LED_SMD:LED_0201_0603Metric -> LED_SMD:LED_0603_1608Metric
- L1: footprint Inductor_SMD:L_0201_0603Metric -> Inductor_SMD:L_0603_1608Metric
- R1, RBOT1, RS1, RTOP1: footprint Resistor_SMD:R_0201_0603Metric -> Resistor_SMD:R_0603_1608Metric
- RCP1: renamed from CPR1; footprint Resistor_SMD:R_0201_0603Metric -> Resistor_SMD:R_0603_1608Metric
- RCP2: renamed from CPR2; footprint Resistor_SMD:R_0201_0603Metric -> Resistor_SMD:R_0603_1608Metric
- RCP3: renamed from CPR3; footprint Resistor_SMD:R_0201_0603Metric -> Resistor_SMD:R_0603_1608Metric
- RCP4: renamed from CPR4; footprint Resistor_SMD:R_0201_0603Metric -> Resistor_SMD:R_0603_1608Metric
- RCP5: renamed from CPR5; footprint Resistor_SMD:R_0201_0603Metric -> Resistor_SMD:R_0603_1608Metric
- RCP6: renamed from CPR6; footprint Resistor_SMD:R_0201_0603Metric -> Resistor_SMD:R_0603_1608Metric
- Y1: footprint Crystal:Crystal_SMD_Abracon_ABM10-4Pin_2.5x2.0mm -> CrystalSMD:Crystal_SMD_NX3225GD

Commit message: Add reference backup layout for 0201 mistake, Resolve issues, & Finish component layout.
Parts:
- removed U3: AT42QT1010-TSHR, Package_TO_SOT_SMD:SOT-23-6, symbol Sensor_Touch:AT42QT1010-TSHR
- added C3: 0.1uF, Capacitor_SMD:C_0603_1608Metric, symbol Device:C
- added U3: AT42QT1010-MAH, AT42QT1010:DFN-8-1EP_2x2mm_P0.5mm_EP0.9x1.5mm, symbol at42qt1010-mah:AT42QT1010-MAH
- BT1: footprint BattHolder:BatteryHolder_LINX_BAT-HLD-001-SMT -> BattHolder:BatteryHolder_LINX_BAT-HLD-001-SMT_SOLDERPAD
- J2: footprint CapSense:CapSense_MaskedPad_D10.0mm -> CapSense:CapSense_MaskedPad_D6.0mm
Connections:
- wire segments 147 -> 146
Changed lines of the file:
@@
 $EndDescr
-$Comp
-L Sensor_Touch:AT42QT1010-TSHR U3
-U 1 1 5B9CB211
-P 1900 6650
-F 0 "U3" H 2050 7000 50  0000 C CNN
-F 1 "AT42QT1010-TSHR" H 2350 6900 50  0000 C CNN
-F 2 "Package_TO_SOT_SMD:SOT-23-6" H 1950 6400 50  0001 L CNN
-F 3 "http://ww1.microchip.com/downloads/en/DeviceDoc/Atmel-9541-AT42-QTouch-BSW-AT42QT1010_Datasheet.pdf" H 2170 7200 50  0001 C CNN
-	1    1900 6650
-	1    0    0    -1
-$EndComp
 $Comp
 L MCU_Microchip_ATmega:ATmega328P-MMH U1
@@
 L Device:R RS1
 U 1 1 5BAB9902
-P 2800 6550
-F 0 "RS1" V 2700 6550 50  0000 C CNN
-F 1 "10K" V 2800 6550 50  0000 C CNN
-F 2 "Resistor_SMD:R_0603_1608Metric" V 2730 6550 50  0001 C CNN
-F 3 "~" H 2800 6550 50  0001 C CNN
-	1    2800 6550
+P 2750 6500
+F 0 "RS1" V 2650 6500 50  0000 C CNN
+F 1 "10K" V 2750 6500 50  0000 C CNN
+F 2 "Resistor_SMD:R_0603_1608Metric" V 2680 6500 50  0001 C CNN
+F 3 "~" H 2750 6500 50  0001 C CNN
+	1    2750 6500
 	0    1    1    0
 $EndComp
@@
 L Device:C CS1
 U 1 1 5BAB9A9B
-P 2450 6700
-F 0 "CS1" H 2565 6746 50  0000 L CNN
-F 1 "22nF" H 2565 6655 50  0000 L CNN
-F 2 "Capacitor_SMD:C_1206_3216Metric_Pad1.42x1.75mm_HandSolder" H 2488 6550 50  0001 C CNN
-F 3 "~" H 2450 6700 50  0001 C CNN
-	1    2450 6700
-	1    0    0    -1
-$EndComp
-Text GLabel 1500 6750 0    50   Output ~ 0
+P 2300 6650
+F 0 "CS1" H 2415 6696 50  0000 L CNN
+F 1 "22nF" H 2415 6605 50  0000 L CNN
+F 2 "Capacitor_SMD:C_1206_3216Metric_Pad1.42x1.75mm_HandSolder" H 2338 6500 50  0001 C CNN
+F 3 "~" H 2300 6650 50  0001 C CNN
+	1    2300 6650
+	1    0    0    -1
+$EndComp
+Text GLabel 1350 6500 0    50   Output ~ 0
 CAPSENSE
-Text GLabel 2300 1400 2    50   Input ~ 0
+Text GLabel 2300 2500 2    50   Input ~ 0
 CAPSENSE
-Wire Wire Line
-	2300 6750 2300 6850
-Wire Wire Line
-	2300 6850 2450 6850
-Wire Wire Line
-	2300 6550 2450 6550
-Wire Wire Line
-	2450 6550 2650 6550
-Connection ~ 2450 6550
-Wire Wire Line
-	2950 6550 3050 6550
-$Comp
-L power:GND #PWR017
+$Comp
+L power:GND #PWR018
 U 1 1 5BAD403F
-P 1900 7050
-F 0 "#PWR017" H 1900 6800 50  0001 C CNN
-F 1 "GND" H 1905 6877 50  0000 C CNN
-F 2 "" H 1900 7050 50  0001 C CNN
-F 3 "" H 1900 7050 50  0001 C CNN
-	1    1900 7050
-	1    0    0    -1
-$EndComp
-Wire Wire Line
-	1900 6950 1900 7050
+P 1750 7100
+F 0 "#PWR018" H 1750 6850 50  0001 C CNN
+F 1 "GND" H 1755 6927 50  0000 C CNN
+F 2 "" H 1750 7100 50  0001 C CNN
+F 3 "" H 1750 7100 50  0001 C CNN
+	1    1750 7100
+	1    0    0    -1
+$EndComp
 $Comp
 L power:+3V3 #PWR015
 U 1 1 5BAD7268
-P 1900 6250
-F 0 "#PWR015" H 1900 6100 50  0001 C CNN
-F 1 "+3V3" H 1915 6423 50  0000 C CNN
-F 2 "" H 1900 6250 50  0001 C CNN
-F 3 "" H 1900 6250 50  0001 C CNN
-	1    1900 6250
-	1    0    0    -1
-$EndComp
-Wire Wire Line
-	1900 6250 1900 6350
-$Comp
-L power:GND #PWR016
+P 1750 6050
+F 0 "#PWR015" H 1750 5900 50  0001 C CNN
+F 1 "+3V3" H 1765 6223 50  0000 C CNN
+F 2 "" H 1750 6050 50  0001 C CNN
+F 3 "" H 1750 6050 50  0001 C CNN
+	1    1750 6050
+	1    0    0    -1
+$EndComp
+$Comp
+L power:GND #PWR017
 U 1 1 5BADA5AF
-P 1350 6450
-F 0 "#PWR016" H 1350 6200 50  0001 C CNN
-F 1 "GND" H 1355 6277 50  0000 C CNN
-F 2 "" H 1350 6450 50  0001 C CNN
-F 3 "" H 1350 6450 50  0001 C CNN
-	1    1350 6450
-	1    0    0    -1
-$EndComp
-Wire Wire Line
-	1350 6450 1500 6450
-Wire Wire Line
-	1500 6450 1500 6550
-Text Notes 1550 7450 0    50   ~ 0
+P 2150 6900
+F 0 "#PWR017" H 2150 6650 50  0001 C CNN
+F 1 "GND" H 2155 6727 50  0000 C CNN
+F 2 "" H 2150 6900 50  0001 C CNN
+F 3 "" H 2150 6900 50  0001 C CNN
+	1    2150 6900
+	1    0    0    -1
+$EndComp
+Text Notes 2550 6950 0    50   ~ 0
 Capacitive Touch Button
 Text Notes 8750 4600 0    50   ~ 0
@@
 F 0 "BT1" H 3768 4646 50  0000 L CNN
 F 1 "CR2032" H 3768 4555 50  0000 L CNN
-F 2 "BattHolder:BatteryHolder_LINX_BAT-HLD-001-SMT" V 3650 4610 50  0001 C CNN
+F 2 "BattHolder:BatteryHolder_LINX_BAT-HLD-001-SMT_SOLDERPAD" V 3650 4610 50  0001 C CNN
 F 3 "~" V 3650 4610 50  0001 C CNN
 	1    3650 4550
@@
 NoConn ~ 2300 2300
 NoConn ~ 2300 2400
-NoConn ~ 2300 2500
+NoConn ~ 2300 1400
 NoConn ~ 2300 2600
 NoConn ~ 2300 2700
@@
 L Connector:Conn_01x01_Female J2
 U 1 1 5BA0484D
-P 3250 6550
-F 0 "J2" H 3278 6576 50  0000 L CNN
-F 1 "SENSE_ELECTRODE" H 3278 6485 50  0000 L CNN
-F 2 "CapSense:CapSense_MaskedPad_D10.0mm" H 3250 6550 50  0001 C CNN
-F 3 "~" H 3250 6550 50  0001 C CNN
-	1    3250 6550
+P 3100 6500
+F 0 "J2" H 3128 6526 50  0000 L CNN
+F 1 "SENSE_ELECTRODE" H 3128 6435 50  0000 L CNN
+F 2 "CapSense:CapSense_MaskedPad_D6.0mm" H 3100 6500 50  0001 C CNN
+F 3 "~" H 3100 6500 50  0001 C CNN
+	1    3100 6500
 	1    0    0    -1
 $EndComp
@@
 	1    0    0    -1
 $EndComp
+$Comp
+L Device:C C3
+U 1 1 5BA0E294
+P 1550 6100
+F 0 "C3" V 1802 6100 50  0000 C CNN
+F 1 "0.1uF" V 1711 6100 50  0000 C CNN
+F 2 "Capacitor_SMD:C_0603_1608Metric" H 1588 5950 50  0001 C CNN
+F 3 "~" H 1550 6100 50  0001 C CNN
+	1    1550 6100
+	0    -1   -1   0
+$EndComp
+$Comp
+L power:GND #PWR016
+U 1 1 5BA22FE2
+P 1400 6100
+F 0 "#PWR016" H 1400 5850 50  0001 C CNN
+F 1 "GND" H 1405 5927 50  0000 C CNN
+F 2 "" H 1400 6100 50  0001 C CNN
+F 3 "" H 1400 6100 50  0001 C CNN
+	1    1400 6100
+	1    0    0    -1
+$EndComp
+Wire Wire Line
+	1750 6300 1750 6100
+Wire Wire Line
+	1700 6100 1750 6100
+Connection ~ 1750 6100
+Wire Wire Line
+	1750 6100 1750 6050
+$Comp
+L at42qt1010-mah:AT42QT1010-MAH U3
+U 1 1 5BA54929
+P 1750 6700
+F 0 "U3" H 1900 7150 50  0000 C CNN
+F 1 "AT42QT1010-MAH" H 2200 7050 50  0000 C CNN
+F 2 "AT42QT1010:DFN-8-1EP_2x2mm_P0.5mm_EP0.9x1.5mm" H 1900 6300 50  0001 L CNN
+F 3 "" H 2020 7250 50  0001 C CNN
+	1    1750 6700
+	1    0    0    -1
+$EndComp
+Wire Wire Line
+	2150 6700 2150 6800
+Wire Wire Line
+	2150 6800 2300 6800
+Wire Wire Line
+	2150 6500 2300 6500
+Wire Wire Line
+	2300 6500 2600 6500
+Connection ~ 2300 6500
+Wire Wire Line
+	1650 7100 1750 7100
+Connection ~ 1750 7100
 $EndSCHEMATC

Commit message: Finish board routing, Add LED Charlieplexing truth table, Add jumpered electrode just in case
Parts:
- added C3: 0.1uF, Capacitor_SMD:C_0603_1608Metric, symbol Device:C
- added J3: SENSE_ELECTRODE_AUX, CapSense:SMD_WIREPAD_4.0x1.25mm, symbol Connector:Conn_01x01_Female
- added JP1: Jumper_NO_Small, Jumper:SolderJumper-2_P1.3mm_Open_RoundedPad1.0x1.5mm, symbol Device:Jumper_NO_Small
- renumbered C3 to C4
Connections:
- wire segments 146 -> 150
Changed lines of the file:
@@
 Connection ~ 9600 1550
-Wire Wire Line
-	10100 1550 10450 1550
-Connection ~ 10100 1550
 Wire Wire Line
 	8200 2150 8600 2150
@@
 Wire Wire Line
 	9950 2150 10100 2150
-Connection ~ 10450 1550
 Wire Wire Line
 	10100 1850 10250 1850
@@
 Connection ~ 10450 2450
 Wire Wire Line
-	10450 2450 10450 1550
-Wire Wire Line
 	10100 3050 10450 3050
 Connection ~ 10450 3050
@@
 Wire Wire Line
 	10450 3650 10450 3050
-Wire Wire Line
-	10450 950  10100 950
-Wire Wire Line
-	10450 950  10450 1550
-Connection ~ 10100 950
 Text GLabel 7900 3350 0    50   3State ~ 0
 CP5
@@
 CP2
 $Comp
-L power:+3V3 #PWR06
+L power:+3V3 #PWR07
 U 1 1 5BA982AE
 P 2950 2900
-F 0 "#PWR06" H 2950 2750 50  0001 C CNN
+F 0 "#PWR07" H 2950 2750 50  0001 C CNN
 F 1 "+3V3" H 2965 3073 50  0000 C CNN
 F 2 "" H 2950 2900 50  0001 C CNN
@@
 $EndComp
 $Comp
-L power:+3V3 #PWR01
+L power:+3V3 #PWR02
 U 1 1 5BAA1804
-P 1750 950
-F 0 "#PWR01" H 1750 800 50  0001 C CNN
-F 1 "+3V3" H 1765 1123 50  0000 C CNN
-F 2 "" H 1750 950 50  0001 C CNN
-F 3 "" H 1750 950 50  0001 C CNN
-	1    1750 950
-	1    0    0    -1
-$EndComp
-Wire Wire Line
-	1700 1100 1700 1050
-Wire Wire Line
-	1800 1100 1800 1050
-Wire Wire Line
-	1700 1050 1750 1050
-Wire Wire Line
-	1750 1050 1750 950
-Wire Wire Line
-	1800 1050 1750 1050
-Connection ~ 1750 1050
-$Comp
-L power:+3V3 #PWR02
+P 1800 1100
+F 0 "#PWR02" H 1800 950 50  0001 C CNN
+F 1 "+3V3" H 1815 1273 50  0000 C CNN
+F 2 "" H 1800 1100 50  0001 C CNN
+F 3 "" H 1800 1100 50  0001 C CNN
+	1    1800 1100
+	1    0    0    -1
+$EndComp
+$Comp
+L power:+3V3 #PWR03
 U 1 1 5BAA9F84
 P 1000 1400
-F 0 "#PWR02" H 1000 1250 50  0001 C CNN
+F 0 "#PWR03" H 1000 1250 50  0001 C CNN
 F 1 "+3V3" H 1015 1573 50  0000 C CNN
 F 2 "" H 1000 1400 50  0001 C CNN
@@
 	1000 1400 1100 1400
 $Comp
-L power:GND #PWR07
+L power:GND #PWR08
 U 1 1 5BAAEA5E
 P 1700 4200
-F 0 "#PWR07" H 1700 3950 50  0001 C CNN
+F 0 "#PWR08" H 1700 3950 50  0001 C CNN
 F 1 "GND" H 1705 4027 50  0000 C CNN
 F 2 "" H 1700 4200 50  0001 C CNN
@@
 	1    0    0    -1
 $EndComp
-Wire Wire Line
-	1700 4200 1700 4100
 $Comp
 L Device:R R1
@@
 Text GLabel 1350 6500 0    50   Output ~ 0
 CAPSENSE
-Text GLabel 2300 2500 2    50   Input ~ 0
+Text GLabel 2300 1400 2    50   Input ~ 0
 CAPSENSE
 $Comp
-L power:GND #PWR018
+L power:GND #PWR019
 U 1 1 5BAD403F
 P 1750 7100
-F 0 "#PWR018" H 1750 6850 50  0001 C CNN
+F 0 "#PWR019" H 1750 6850 50  0001 C CNN
 F 1 "GND" H 1755 6927 50  0000 C CNN
 F 2 "" H 1750 7100 50  0001 C CNN
@@
 $EndComp
 $Comp
-L power:+3V3 #PWR015
+L power:+3V3 #PWR016
 U 1 1 5BAD7268
 P 1750 6050
-F 0 "#PWR015" H 1750 5900 50  0001 C CNN
+F 0 "#PWR016" H 1750 5900 50  0001 C CNN
 F 1 "+3V3" H 1765 6223 50  0000 C CNN
 F 2 "" H 1750 6050 50  0001 C CNN
@@
 $EndComp
 $Comp
-L power:GND #PWR017
+L power:GND #PWR018
 U 1 1 5BADA5AF
 P 2150 6900
-F 0 "#PWR017" H 2150 6650 50  0001 C CNN
+F 0 "#PWR018" H 2150 6650 50  0001 C CNN
 F 1 "GND" H 2155 6727 50  0000 C CNN
 F 2 "" H 2150 6900 50  0001 C CNN
@@
 	1    0    0    -1
 $EndComp
-Text Notes 2550 6950 0    50   ~ 0
+Text Notes 2350 7250 0    50   ~ 0
 Capacitive Touch Button
 Text Notes 8750 4600 0    50   ~ 0
@@
 	2950 2300 2950 2350
 $Comp
-L power:GND #PWR04
+L power:GND #PWR05
 U 1 1 5BB2FCCB
 P 2950 2350
-F 0 "#PWR04" H 2950 2100 50  0001 C CNN
+F 0 "#PWR05" H 2950 2100 50  0001 C CNN
 F 1 "GND" H 2955 2177 50  0000 C CNN
 F 2 "" H 2950 2350 50  0001 C CNN
@@
 $EndComp
 $Comp
-L power:GND #PWR012
+L power:GND #PWR013
 U 1 1 5BB3B3F5
 P 4950 5000
-F 0 "#PWR012" H 4950 4750 50  0001 C CNN
+F 0 "#PWR013" H 4950 4750 50  0001 C CNN
 F 1 "GND" H 4955 4827 50  0000 C CNN
 F 2 "" H 4950 5000 50  0001 C CNN
@@
 $EndComp
 $Comp
-L power:GND #PWR010
+L power:GND #PWR011
 U 1 1 5BB468E0
 P 4200 4650
-F 0 "#PWR010" H 4200 4400 50  0001 C CNN
+F 0 "#PWR011" H 4200 4400 50  0001 C CNN
 F 1 "GND" H 4205 4477 50  0000 C CNN
 F 2 "" H 4200 4650 50  0001 C CNN
@@
 	4600 4350 4650 4350
 $Comp
-L power:GND #PWR09
+L power:GND #PWR010
 U 1 1 5BB5585E
 P 3650 4650
-F 0 "#PWR09" H 3650 4400 50  0001 C CNN
+F 0 "#PWR010" H 3650 4400 50  0001 C CNN
 F 1 "GND" H 3655 4477 50  0000 C CNN
 F 2 "" H 3650 4650 50  0001 C CNN
@@
 $EndComp
 $Comp
-L power:GND #PWR011
+L power:GND #PWR012
 U 1 1 5BB6CE63
 P 6200 4750
-F 0 "#PWR011" H 6200 4500 50  0001 C CNN
+F 0 "#PWR012" H 6200 4500 50  0001 C CNN
 F 1 "GND" H 6205 4577 50  0000 C CNN
 F 2 "" H 6200 4750 50  0001 C CNN
@@
 Connection ~ 5750 4450
 $Comp
-L power:+3V3 #PWR08
+L power:+3V3 #PWR09
 U 1 1 5BB7F37F
 P 6200 4450
-F 0 "#PWR08" H 6200 4300 50  0001 C CNN
+F 0 "#PWR09" H 6200 4300 50  0001 C CNN
 F 1 "+3V3" H 6215 4623 50  0000 C CNN
 F 2 "" H 6200 4450 50  0001 C CNN
@@
 	5750 4800 5750 4850
 $Comp
-L power:GND #PWR014
+L power:GND #PWR015
 U 1 1 5BB8C362
 P 5750 5150
-F 0 "#PWR014" H 5750 4900 50  0001 C CNN
+F 0 "#PWR015" H 5750 4900 50  0001 C CNN
 F 1 "GND" H 5755 4977 50  0000 C CNN
 F 2 "" H 5750 5150 50  0001 C CNN
@@
 $EndComp
 $Comp
-L power:GND #PWR013
+L power:GND #PWR014
 U 1 1 5BB8C492
 P 5150 5000
-F 0 "#PWR013" H 5150 4750 50  0001 C CNN
+F 0 "#PWR014" H 5150 4750 50  0001 C CNN
 F 1 "GND" H 5155 4827 50  0000 C CNN
 F 2 "" H 5150 5000 50  0001 C CNN
@@
 NoConn ~ 2300 2300
 NoConn ~ 2300 2400
-NoConn ~ 2300 1400
+NoConn ~ 2300 2500
 NoConn ~ 2300 2600
 NoConn ~ 2300 2700
@@
 Programming Pads
 $Comp
-L power:GND #PWR05
+L power:GND #PWR06
 U 1 1 5BBFA6C8
 P 5050 2450
-F 0 "#PWR05" H 5050 2200 50  0001 C CNN
+F 0 "#PWR06" H 5050 2200 50  0001 C CNN
 F 1 "GND" H 5055 2277 50  0000 C CNN
 F 2 "" H 5050 2450 50  0001 C CNN
@@
 $EndComp
 $Comp
-L power:+3V3 #PWR03
+L power:+3V3 #PWR04
 U 1 1 5BBFA83F
 P 5050 1550
-F 0 "#PWR03" H 5050 1400 50  0001 C CNN
+F 0 "#PWR04" H 5050 1400 50  0001 C CNN
 F 1 "+3V3" H 5065 1723 50  0000 C CNN
 F 2 "" H 5050 1550 50  0001 C CNN
@@
 L Connector:Conn_01x01_Female J2
 U 1 1 5BA0484D
-P 3100 6500
-F 0 "J2" H 3128 6526 50  0000 L CNN
-F 1 "SENSE_ELECTRODE" H 3128 6435 50  0000 L CNN
-F 2 "CapSense:CapSense_MaskedPad_D6.0mm" H 3100 6500 50  0001 C CNN
-F 3 "~" H 3100 6500 50  0001 C CNN
-	1    3100 6500
+P 3200 6500
+F 0 "J2" H 3228 6526 50  0000 L CNN
+F 1 "SENSE_ELECTRODE" H 3228 6435 50  0000 L CNN
+F 2 "CapSense:CapSense_MaskedPad_D6.0mm" H 3200 6500 50  0001 C CNN
+F 3 "~" H 3200 6500 50  0001 C CNN
+	1    3200 6500
 	1    0    0    -1
 $EndComp
@@
 $EndComp
 $Comp
-L Device:C C3
+L Device:C C4
 U 1 1 5BA0E294
 P 1550 6100
-F 0 "C3" V 1802 6100 50  0000 C CNN
+F 0 "C4" V 1802 6100 50  0000 C CNN
 F 1 "0.1uF" V 1711 6100 50  0000 C CNN
 F 2 "Capacitor_SMD:C_0603_1608Metric" H 1588 5950 50  0001 C CNN
@@
 $EndComp
 $Comp
-L power:GND #PWR016
+L power:GND #PWR017
 U 1 1 5BA22FE2
 P 1400 6100
-F 0 "#PWR016" H 1400 5850 50  0001 C CNN
+F 0 "#PWR017" H 1400 5850 50  0001 C CNN
 F 1 "GND" H 1405 5927 50  0000 C CNN
 F 2 "" H 1400 6100 50  0001 C CNN
@@
 	1650 7100 1750 7100
 Connection ~ 1750 7100
+$Comp
+L Connector:Conn_01x01_Female J3
+U 1 1 5BA3B34E
+P 3150 6900
+F 0 "J3" H 3178 6926 50  0000 L CNN
+F 1 "SENSE_ELECTRODE_AUX" H 3178 6835 50  0000 L CNN
+F 2 "CapSense:SMD_WIREPAD_4.0x1.25mm" H 3150 6900 50  0001 C CNN
+F 3 "~" H 3150 6900 50  0001 C CNN
+	1    3150 6900
+	1    0    0    -1
+$EndComp
+Wire Wire Line
+	2900 6500 2950 6500
+$Comp
+L Device:Jumper_NO_Small JP1
+U 1 1 5BAA0B06
+P 2950 6700
+F 0 "JP1" V 2904 6748 50  0000 L CNN
+F 1 "Jumper_NO_Small" V 2995 6748 50  0000 L CNN
+F 2 "Jumper:SolderJumper-2_P1.3mm_Open_RoundedPad1.0x1.5mm" H 2950 6700 50  0001 C CNN
+F 3 "~" H 2950 6700 50  0001 C CNN
+	1    2950 6700
+	0    1    1    0
+$EndComp
+Wire Wire Line
+	2950 6500 2950 6600
+Connection ~ 2950 6500
+Wire Wire Line
+	2950 6500 3000 6500
+Wire Wire Line
+	2950 6800 2950 6900
+$Comp
+L Device:C C3
+U 1 1 5BAB7CFE
+P 900 2450
+F 0 "C3" V 850 2550 50  0000 C CNN
+F 1 "0.1uF" V 1050 2450 50  0000 C CNN
+F 2 "Capacitor_SMD:C_0603_1608Metric" H 938 2300 50  0001 C CNN
+F 3 "~" H 900 2450 50  0001 C CNN
+	1    900  2450
+	-1   0    0    1
+$EndComp
+$Comp
+L power:+3V3 #PWR01
+U 1 1 5BAB810C
+P 1700 1000
+F 0 "#PWR01" H 1700 850 50  0001 C CNN
+F 1 "+3V3" H 1715 1173 50  0000 C CNN
+F 2 "" H 1700 1000 50  0001 C CNN
+F 3 "" H 1700 1000 50  0001 C CNN
+	1    1700 1000
+	1    0    0    -1
+$EndComp
+Wire Wire Line
+	1700 1100 1700 1050
+Wire Wire Line
+	1700 1050 900  1050
+Wire Wire Line
+	900  1050 900  2300
+Connection ~ 1700 1050
+Wire Wire Line
+	1700 1050 1700 1000
+Wire Wire Line
+	1700 4100 1700 4150
+Wire Wire Line
+	1700 4150 900  4150
+Wire Wire Line
+	900  2600 900  4150
+Connection ~ 1700 4150
+Wire Wire Line
+	1700 4150 1700 4200
+Wire Wire Line
+	10450 2450 10450 1550
+Connection ~ 10100 1550
+Wire Wire Line
+	10100 1550 10450 1550
 $EndSCHEMATC

Commit message: Finalize PCB, Generate drill files for manufacturing, Begin lasercut enclosure design
Parts:
- J1: footprint Connector_PinHeader_2.54mm:PinHeader_1x06_P2.54mm_Vertical -> ISP_Connector:SIP-6_AVR_ISP
Other:
- note added: "32KHz Watch for Timekeeping"
- note added: "Crystal Value May Change to"
Changed lines of the file:
@@
 F 0 "J1" H 4870 2146 50  0000 R CNN
 F 1 "AVR-ISP-6" H 4870 2055 50  0000 R CNN
-F 2 "Connector_PinHeader_2.54mm:PinHeader_1x06_P2.54mm_Vertical" V 4900 2100 50  0001 C CNN
+F 2 "ISP_Connector:SIP-6_AVR_ISP" V 4900 2100 50  0001 C CNN
 F 3 " ~" H 3875 1500 50  0001 C CNN
 	1    5150 2050
@@
 Wire Wire Line
 	10100 1550 10450 1550
+Text Notes 3000 2100 0    50   ~ 0
+Crystal Value May Change to
+Text Notes 3000 2200 0    50   ~ 0
+32KHz Watch for Timekeeping
 $EndSCHEMATC
